Commit message: *

File: src/quadrobot_viewer/urdf/quadrobot.urdf (robot description, URDF)
Before this commit: robot quadrobot, 15 links, 14 joints
Links:
- link BLA: mass 0.0109452431127404 -> 0.010945
- link FLA: mass 0.010945 -> 0.0109452431127404
Joints:
- joint joint_BLA: origin xyz=0.03 0.055 0.005 rpy=1.5708 -0.0079223 3.1416 -> xyz=0.03 -0.055 0.005 rpy=-1.5708 0.0092604 -3.1416
- joint joint_BLB: origin xyz=-0.040001 0 0.01 rpy=-1.5708 -0.28877 1.5708 -> xyz=-0.039319 0 0.01 rpy=-1.5708 0.35696 1.5708
- joint joint_BLC: origin xyz=0 -0.1 0.01 rpy=0 0 -1.2863 -> xyz=0 -0.1 0.0094885 rpy=0 0 1.1668
- joint joint_BRA: origin xyz=-0.03 0.055 0.005 rpy=-1.5708 0.040291 0 -> xyz=-0.03 -0.055 0.005 rpy=1.5708 0.022451 0
- joint joint_BRB: origin xyz=-0.040016 0 0.01 rpy=-1.5708 -0.33726 -1.5708 -> xyz=-0.040005 0 0.01 rpy=-1.5708 0.33034 -1.5708
- joint joint_BRC: origin xyz=0 -0.1 -0.01 rpy=0 0 -1.2397 -> xyz=0 -0.1 -0.01 rpy=0 0 1.2033
- joint joint_FLA: origin xyz=0.03 -0.055 0.005 rpy=-1.5708 0.0092604 -3.1416 -> xyz=0.03 0.055 0.005 rpy=1.5708 -0.0079223 3.1416
- joint joint_FLB: origin xyz=-0.039319 0 0.01 rpy=-1.5708 0.35696 1.5708 -> xyz=-0.040001 0 0.01 rpy=-1.5708 -0.28877 1.5708
- joint joint_FLC: origin xyz=0 -0.1 0.0094885 rpy=0 0 1.1668 -> xyz=0 -0.1 0.01 rpy=0 0 -1.2863
- joint joint_FRA: origin xyz=-0.03 -0.055 0.005 rpy=1.5708 0.022451 0 -> xyz=-0.03 0.055 0.005 rpy=-1.5708 0.040291 0
- joint joint_FRB: origin xyz=-0.040005 0 0.01 rpy=-1.5708 0.33034 -1.5708 -> xyz=-0.040016 0 0.01 rpy=-1.5708 -0.33726 -1.5708
- joint joint_FRC: origin xyz=0 -0.1 -0.01 rpy=0 0 1.2033 -> xyz=0 -0.1 -0.01 rpy=0 0 -1.2397
