Commit message: Connexion gazebo

File: src/quadrobot_viewer/urdf/quadrobot.ros2_control.xacro (robot description, xacro)
@@ -11,6 +11,6 @@
     </xacro:macro>
     <!-- Macro for ros2_control -->
-    <xacro:macro name="MACRO_QUADROBOT_ROS2_CONTROL" params="hardware_plugin">
-        <ros2_control name="quadrobot.ros2_control" type="system">
+    <xacro:macro name="MACRO_QUADROBOT_ROS2_CONTROL" params="hardware_name hardware_plugin">
+        <ros2_control name="${hardware_name}" type="system">
             <hardware>
                 <plugin>${hardware_plugin}</plugin>

File: src/quadrobot_viewer/urdf/quadrobot.urdf.xacro (robot description, xacro)
@@ -2,4 +2,5 @@
 <robot name="quadrobot" xmlns:xacro="http://www.ros.org/wiki/xacro">
     <!-- Define arguments with default values -->
+    <xacro:arg name="hardware_name" default="GazeboSimSystem" />
     <xacro:arg name="hardware_plugin" default="gz_ros2_control/GazeboSimSystem" />
     <xacro:arg name="config_ros2_control_path"
@@ -9,11 +10,11 @@
     <xacro:include filename="$(find quadrobot_viewer)/urdf/quadrobot.ros2_control.xacro" />
     <!-- Using the MACRO_QUADROBOT_ROS2_CONTROL -->
-    <xacro:MACRO_QUADROBOT_ROS2_CONTROL hardware_plugin="$(arg hardware_plugin)" />
+    <xacro:MACRO_QUADROBOT_ROS2_CONTROL hardware_name="$(arg hardware_name)"
+        hardware_plugin="$(arg hardware_plugin)" />
     <!-- Using Plugin for Gazebo -->
     <gazebo>
         <plugin filename="libgz_ros2_control-system.so"
             name="gz_ros2_control::GazeboSimROS2ControlPlugin">
-            <robot>/robot>
-            <!-- <parameters>$(arg config_ros2_control_path)</parameters> -->
+            <parameters>$(arg config_ros2_control_path)</parameters>
         </plugin>
     </gazebo>
