Commit message: *

File: src/dgz_viewer/urdf/champ.ros2_control.xacro (robot description, xacro)
@@ -9,4 +9,12 @@
             </state_interface>
         </joint>
+    </xacro:macro>
+    <!-- Macro for sensor -->
+    <xacro:macro name="MACRO_SENSOR" params="name">
+        <sensor name="${name}">
+            <state_interface name="position" />
+            <state_interface name="angular_velocity" />
+            <state_interface name="linear_acceleration" />
+        </sensor>
     </xacro:macro>
     <!-- Macro for ros2_control -->
@@ -29,4 +37,6 @@
             <xacro:MACRO_JOINT name="rh_upper_leg_joint" initial_position="0.0" />
             <xacro:MACRO_JOINT name="rh_lower_leg_joint" initial_position="0.0" />
+            <!-- Using the MACRO_SENSOR -->
+            <!-- <xacro:MACRO_SENSOR name="imu_sensor" /> -->
         </ros2_control>
     </xacro:macro>

File: src/dgz_viewer/urdf/champ.urdf.xacro (robot description, xacro)
@@ -48,5 +48,5 @@
     </gazebo>
     <xacro:include filename="$(find dgz_viewer)/urdf/leg.urdf.xacro" />
-    <xacro:include filename="$(find dgz_viewer)/urdf/sensors.xacro" />
+    <!-- <xacro:include filename="$(find dgz_viewer)/urdf/sensors.xacro" /> -->
     <!-- <xacro:include filename="$(find dgz_viewer)/urdf/accessories.urdf.xacro" />
     <xacro:accessories
@@ -84,11 +84,47 @@
     </gazebo> -->
     <!-- ....................................................................... -->
+    <!-- IMU Sensor -->
+    <!-- <link name="imu_sensor_link">
+        <visual>
+            <origin xyz="0 0 0" rpy="0 0 0" />
+            <geometry>
+                <box size="0.02 0.02 0.005" />
+            </geometry>
+            <material name="black">
+                <color rgba="0 0 0 1.0" />
+            </material>
+        </visual>
+    </link>
+    <joint name="imu_sensor_joint" type="fixed">
+        <parent link="base_link" />
+        <child link="imu_sensor_link" />
+        <origin xyz="0 0 0.1" rpy="0 0 0" />
+    </joint>
+    <gazebo reference="imu_sensor_link">
+        <sensor name="imu_sensor" type="imu">
+            <always_on>true</always_on>
+            <update_rate>100</update_rate>
+            <visualize>true</visualize>
+            <topic>/imu_sensor/imu</topic>
+        </sensor>
+    </gazebo> -->
+    <!-- <plugin filename="gz-sim-imu-system"
+        name="gz::sim::systems::Imu">
+    </plugin> -->
+    <!-- <gazebo>
+        <plugin filename="libgazebo_ros_imu_sensor.so" name="imu_sensor">
+            <robotNamespace>dgz</robotNamespace>
+            <topicName>imu/data</topicName>
+            <frameName>imu_link</frameName>
+            <gaussianNoise>0.01</gaussianNoise>
+        </plugin>
+    </gazebo> -->
+    <!-- -->
     <!-- Define arguments with default values -->
     <xacro:arg name="hardware_name" default="GazeboSimSystem" />
     <xacro:arg name="hardware_plugin" default="gz_ros2_control/GazeboSimSystem" />
     <xacro:arg name="config_ros2_control_path"
-        default="$(find dgz_viewer)/config/ros2_control.yaml" />
+        default=" $(find dgz_viewer)/config/ros2_control.yaml" />
     <!-- Include the xacro files -->
-    <!-- <xacro:include filename="$(find dgz_viewer)/urdf/champ.xacro" /> -->
     <xacro:include filename="$(find dgz_viewer)/urdf/champ.ros2_control.xacro" />
     <!-- Using the MACRO_QUADROBOT_ROS2_CONTROL -->

Commit message: Urdfxacro

File: src/dgz_viewer/urdf/champ.ros2_control.xacro (robot description, xacro)
@@ -13,7 +13,17 @@
     <xacro:macro name="MACRO_SENSOR" params="name">
         <sensor name="${name}">
-            <state_interface name="position" />
-            <state_interface name="angular_velocity" />
-            <state_interface name="linear_acceleration" />
+            <!-- State interface orientation -->
+            <state_interface name="orientation.x" />
+            <state_interface name="orientation.y" />
+            <state_interface name="orientation.z" />
+            <state_interface name="orientation.w" />
+            <!-- State interface angular_velocity -->
+            <state_interface name="angular_velocity.x" />
+            <state_interface name="angular_velocity.y" />
+            <state_interface name="angular_velocity.z" />
+            <!-- State interface linear_acceleration -->
+            <state_interface name="linear_acceleration.x" />
+            <state_interface name="linear_acceleration.y" />
+            <state_interface name="linear_acceleration.z" />
         </sensor>
     </xacro:macro>
@@ -38,5 +48,5 @@
             <xacro:MACRO_JOINT name="rh_lower_leg_joint" initial_position="0.0" />
             <!-- Using the MACRO_SENSOR -->
-            <!-- <xacro:MACRO_SENSOR name="imu_sensor" /> -->
+            <xacro:MACRO_SENSOR name="imu_sensor" />
         </ros2_control>
     </xacro:macro>

File: src/dgz_viewer/urdf/champ.urdf.xacro (robot description, xacro)
@@ -85,5 +85,5 @@
     <!-- ....................................................................... -->
     <!-- IMU Sensor -->
-    <!-- <link name="imu_sensor_link">
+    <link name="imu_sensor_link">
         <visual>
             <origin xyz="0 0 0" rpy="0 0 0" />
@@ -108,16 +108,9 @@
             <topic>/imu_sensor/imu</topic>
         </sensor>
-    </gazebo> -->
-    <!-- <plugin filename="gz-sim-imu-system"
-        name="gz::sim::systems::Imu">
-    </plugin> -->
-    <!-- <gazebo>
-        <plugin filename="libgazebo_ros_imu_sensor.so" name="imu_sensor">
-            <robotNamespace>dgz</robotNamespace>
-            <topicName>imu/data</topicName>
-            <frameName>imu_link</frameName>
-            <gaussianNoise>0.01</gaussianNoise>
-        </plugin>
-    </gazebo> -->
+    </gazebo>
+    <gazebo>
+        <plugin filename="gz-sim-imu-system"
+            name="gz::sim::systems::Imu" />
+    </gazebo>
     <!-- -->
     <!-- Define arguments with default values -->
